Commit message: Modify urdf to add world prefix
Signed-off-by: Artur Kamieniecki <artur.kamieniecki@robotec.ai>

File: ros2_ws/src/Universal_Robots_ROS2_Description/urdf/ur.urdf.xacro (robot description, xacro)
@@ -47,10 +47,10 @@
    <xacro:property name="initial_positions_file" default="$(arg initial_positions_file)"/>
    <!-- create link fixed to the "world" -->
-   <link name="world" />
+   <link name="$(arg tf_prefix)world" />
    <!-- arm -->
    <xacro:ur_robot
      name="$(arg name)"
      tf_prefix="$(arg tf_prefix)"
-     parent="world"
+     parent="$(arg tf_prefix)world"
      joint_limits_parameters_file="$(arg joint_limit_params)"
      kinematics_parameters_file="$(arg kinematics_params)"
