Commit message: add gripper to ur20
Signed-off-by: Anna Faferek <anna.faferek@robotec.ai>

File: ros2_ws/src/UR20_moveit_config/config/ur20.urdf (robot description, URDF)
Before this commit: robot ur20, 13 links, 12 joints
Links:
- added link gripper_link; collision mesh filename=package://ur_description/meshes/ur20/collision/Gripper.stl; visual mesh filename=package://ur_description/meshes/ur20/visual/Gripper.dae
Joints:
- added joint tool0-gripper: type fixed, parent tool0, child gripper_link, origin xyz=0 0 0.03 rpy=1.5707963267948966 1.5707963267948966 0
