Commit message: Import robot model

File: ros2_ws/src/OTTO600_Description/Urdf/OTTO600.urdf.xacro (robot description, xacro)
@@ -11,4 +11,7 @@
   <xacro:property name="wheel_length" value="0.11" />
   <xacro:property name="wheel_z_position" value="0.0877" />
+  <xacro:property name="camera_height" value="0.115" />
+  <xacro:property name="camera_center_offset" value="0.05" />
+  <xacro:property name="lidar_height" value="0.2" />
   <link name="base_link">
     <inertial>
@@ -18,5 +21,5 @@
     </inertial>
     <visual>
-      <origin rpy="0. 0. 0." xyz="0. 0. 0."/>
+      <origin rpy="0. 0. ${pi}" xyz="0. 0. 0."/>
       <geometry>
         <mesh filename="../Meshes/OTTO600_bodylink.stl" scale="1.0 1.0 1.0" />
@@ -24,7 +27,7 @@
     </visual>
     <collision>
-      <origin rpy="0. 0. ${pi/2}" xyz="0. 0. ${base_link_height/2 + ground_clearence}"/>
-      <geometry>
-        <box size="${base_link_width} ${base_link_length} ${base_link_height*(1 - ground_clearence)}" />
+      <origin rpy="0. 0. ${pi / 2}" xyz="0. 0. ${base_link_height / 2 + ground_clearence}"/>
+      <geometry>
+        <box size="${base_link_width} ${base_link_length} ${base_link_height * (1 - ground_clearence)}" />
       </geometry>
     </collision>
@@ -230,3 +233,27 @@
     <limit lower="0.0" upper="0.05" effort="0.0" velocity="0.0"/>
   </joint>
+  <link name="lidar_F" />
+  <joint name="lidar_F_joint" type="fixed">
+    <parent link="base_link" />
+    <child link="lidar_F" />
+    <origin rpy="0. 0. 0." xyz="${base_link_length / 2} ${base_link_width / 2} ${lidar_height}" />
+  </joint>
+  <link name="lidar_R" />
+  <joint name="lidar_R_joint" type="fixed">
+    <parent link="base_link" />
+    <child link="lidar_R" />
+    <origin rpy="0. 0. 0." xyz="${-base_link_length / 2} ${-base_link_width / 2} ${lidar_height}" />
+  </joint>
+  <link name="camera_FL" />
+  <joint name="camera_FL_joint" type="fixed">
+    <parent link="base_link" />
+    <child link="camera_FL" />
+    <origin rpy="0. 0. 0." xyz="${base_link_length / 2} ${camera_center_offset} ${camera_height}" />
+  </joint>
+  <link name="camera_FR" />
+  <joint name="camera_FR_joint" type="fixed">
+    <parent link="base_link" />
+    <child link="camera_FR" />
+    <origin rpy="0. 0. 0." xyz="${base_link_length / 2} ${-camera_center_offset} ${camera_height}" />
+  </joint>
 </robot>

Commit message: Add lifting module steering
Signed-off-by: Anna Faferek <anna.faferek@robotec.ai>

File: ros2_ws/src/OTTO600_Description/Urdf/OTTO600.urdf.xacro (robot description, xacro)
@@ -231,5 +231,5 @@
     <axis xyz="0. 0. 1." />
     <origin rpy="0. 0. 0." xyz="0. 0. 0." />
-    <limit lower="0.0" upper="0.05" effort="0.0" velocity="0.0"/>
+    <limit lower="0.0" upper="0.045" effort="0.0" velocity="0.0"/>
   </joint>
   <link name="lidar_F" />

Commit message: Change colliders in urdf
Signed-off-by: Anna Faferek <anna.faferek@robotec.ai>

File: ros2_ws/src/OTTO600_Description/Urdf/OTTO600.urdf.xacro (robot description, xacro)
@@ -3,6 +3,4 @@
  <xacro:property name="base_link_length" value="1.05" />
   <xacro:property name="base_link_width" value="0.697" />
-  <xacro:property name="base_link_height" value="0.289" />
-  <xacro:property name="ground_clearence" value="0.03" />
   <xacro:property name="wheel_axis_front" value="0.406" />
   <xacro:property name="wheel_axis_rear" value="-0.406" />
@@ -26,8 +24,23 @@
       </geometry>
     </visual>
-    <collision>
-      <origin rpy="0. 0. ${pi / 2}" xyz="0. 0. ${base_link_height / 2 + ground_clearence}"/>
-      <geometry>
-        <box size="${base_link_width} ${base_link_length} ${base_link_height * (1 - ground_clearence)}" />
+    <!-- bottom collider box -->
+    <collision>
+      <origin rpy="0. 0. ${pi / 2}" xyz="0. 0. 0.264"/>
+      <geometry>
+        <box size="${base_link_width} ${base_link_length} 0.114" />
+      </geometry>
+    </collision>
+    <!-- center collider box -->
+    <collision>
+      <origin rpy="0. 0. ${pi / 2}" xyz="0. 0. 0.192"/>
+      <geometry>
+        <box size="0.56 0.88 0.03" />
+      </geometry>
+    </collision>
+    <!-- top collider box -->
+    <collision>
+      <origin rpy="0. 0. ${pi / 2}" xyz="0. 0. 0.103"/>
+      <geometry>
+        <box size="${base_link_width} ${base_link_length} 0.145" />
       </geometry>
     </collision>
