Commit message: import new model and add lidar

File: ros2_ws/src/OTTO1500_Description/urdf/OTTO1500_basic_platform.urdf.xacro (robot description, xacro)
@@ -13,15 +13,9 @@
   <xacro:property name="wheel_center_radius" value="0.147" />
   <xacro:property name="wheel_center_length" value="0.1" />
-  <xacro:property name="lift_base_width" value="1." />
-  <xacro:property name="lift_base_length" value="1.35" />
-  <xacro:property name="lift_base_height" value="0.14" />
-  <xacro:property name="lift_base_offset" value="0.04" />
-  <xacro:property name="lift_base_collider_offset" value="0.07" />
-  <xacro:property name="lift_upper_width" value="0.5" />
-  <xacro:property name="lift_upper_length" value="1.2" />
-  <xacro:property name="lift_upper_height" value="0.02" />
-  <xacro:property name="upper_lift_limit" value="0.3" />
-  <xacro:property name="lift_module_height" value="0.14" />
-  <xacro:property name="lift_module_offset" value="0.02" />
+  <xacro:property name="basic_platform_width" value="0.963" />
+  <xacro:property name="basic_platform_length" value="1.53" />
+  <xacro:property name="basic_platform_height" value="0.015" />
+  <xacro:property name="basic_platform_offset" value="0.376" />
+  <xacro:property name="basic_platform_collider_offset" value="0.005" />
   <xacro:property name="camera_height" value="0.22" />
   <xacro:property name="camera_center_offset" value="0.51" />
@@ -197,5 +191,5 @@
     <origin rpy="0. 0. 0." xyz="${wheel_axis_rear} ${-wheel_track} ${wheel_front_rear_radius}" />
   </joint>
-  <link name="lifting_platform_base">
+  <link name="basic_platform">
     <inertial>
       <origin xyz="0. 0. 0." />
@@ -204,13 +198,13 @@
     </inertial>
     <visual>
-      <origin rpy="0. 0. ${pi/2}" xyz="0. 0. ${base_link_height + lift_base_offset}"/>
-      <geometry>
-        <mesh filename="../meshes/Platform_B.stl" scale="1.0 1.0 1.0" />
+      <origin rpy="0. 0. ${pi/2}" xyz="0. 0. ${basic_platform_offset}"/>
+      <geometry>
+        <mesh filename="../meshes/Platform_A.stl" scale="1.0 1.0 1.0" />
       </geometry>
     </visual>
     <collision>=
-      <origin rpy="0. 0. ${pi/2}" xyz="0. 0. ${base_link_height + lift_base_offset + lift_base_collider_offset}"/>
-      <geometry>
-        <box size="${lift_base_width} ${lift_base_length} ${lift_base_height}" />
+      <origin rpy="0. 0. ${pi/2}" xyz="0. 0. ${basic_platform_offset + basic_platform_collider_offset}"/>
+      <geometry>
+        <box size="${basic_platform_width} ${basic_platform_length} ${basic_platform_height}" />
       </geometry>
     </collision>
@@ -218,50 +212,6 @@
   <joint name="platform_base_joint" type="fixed">
     <parent link="base_link" />
-    <child link="lifting_platform_base" />
+    <child link="basic_platform" />
     <origin rpy="0. 0. 0." xyz="0. 0. 0." />
-  </joint>
-  <link name="lift_module">
-    <inertial>
-      <origin xyz="0. 0. 0." />
-      <mass value="15" />
-      <inertia ixx="1." ixy="0." ixz="0." iyy="1." iyz="0." izz="1."/>
-    </inertial>
-    <visual>
-      <origin rpy="0. 0. ${pi/2}" xyz="0. 0. 0."/>
-      <geometry>
-        <mesh filename="../meshes/lift.stl" scale="1.0 1.0 1.0" />
-      </geometry>
-    </visual>
-  </link>
-  <joint name="lift_module_joint" type="fixed">
-    <parent link="base_link" />
-    <child link="lift_module" />
-    <origin rpy="0. 0. 0." xyz="0. 0. ${base_link_height + lift_base_offset + lift_module_offset}" />
-  </joint>
-  <link name="lift_upper">
-    <inertial>
-      <origin xyz="0. 0. 0." />
-      <mass value="15" />
-      <inertia ixx="1." ixy="0." ixz="0." iyy="1." iyz="0." izz="1."/>
-    </inertial>
-    <visual>
-      <origin rpy="0. 0. ${pi/2}" xyz="0. 0. ${base_link_box_height + lift_module_height}"/>
-      <geometry>
-        <mesh filename="../meshes/lift_upper.stl" scale="1.0 1.0 1.0" />
-      </geometry>
-    </visual>
-    <collision>
-      <origin rpy="0. 0. ${pi/2}" xyz="0. 0. ${base_link_box_height + lift_module_height}"/>
-      <geometry>
-        <box size="${lift_upper_width} ${lift_upper_length} ${lift_upper_height}" />
-      </geometry>
-    </collision>
-  </link>
-  <joint name="lift_upper_joint" type="prismatic">
-    <parent link="base_link" />
-    <child link="lift_upper" />
-    <axis xyz="0. 0. 1." />
-    <origin rpy="0. 0. 0." xyz="0. 0. 0." />
-    <limit lower="0.0" upper="${upper_lift_limit}" effort="0.0" velocity="0.0"/>
   </joint>
   <link name="lidar_F" />

Commit message: Add lidars and  lift module to otto1500. Split robot model into two different ones based on platform. (#62)
* Add lift to otto1500 urdf
* import new model and add lidar
* Add collider inside prefab
* Change colliders in urdf
* decrease points per layer number in lidar for better performance and change lidar angle to 270

Signed-off-by: Anna Faferek <anna.faferek@robotec.ai>

---------

Signed-off-by: Anna Faferek <anna.faferek@robotec.ai>

File: ros2_ws/src/OTTO1500_Description/urdf/OTTO1500_basic_platform.urdf.xacro (robot description, xacro)
@@ -12,15 +12,9 @@
   <xacro:property name="wheel_center_radius" value="0.147" />
   <xacro:property name="wheel_center_length" value="0.1" />
-  <xacro:property name="lift_base_width" value="1." />
-  <xacro:property name="lift_base_length" value="1.35" />
-  <xacro:property name="lift_base_height" value="0.14" />
-  <xacro:property name="lift_base_offset" value="0.04" />
-  <xacro:property name="lift_base_collider_offset" value="0.07" />
-  <xacro:property name="lift_upper_width" value="0.5" />
-  <xacro:property name="lift_upper_length" value="1.2" />
-  <xacro:property name="lift_upper_height" value="0.02" />
-  <xacro:property name="upper_lift_limit" value="0.3" />
-  <xacro:property name="lift_module_height" value="0.14" />
-  <xacro:property name="lift_module_offset" value="0.02" />
+  <xacro:property name="basic_platform_width" value="0.963" />
+  <xacro:property name="basic_platform_length" value="1.53" />
+  <xacro:property name="basic_platform_height" value="0.015" />
+  <xacro:property name="basic_platform_offset" value="0.376" />
+  <xacro:property name="basic_platform_collider_offset" value="0.005" />
   <xacro:property name="camera_height" value="0.22" />
   <xacro:property name="camera_center_offset" value="0.51" />
@@ -211,5 +205,5 @@
     <origin rpy="0. 0. 0." xyz="${wheel_axis_rear} ${-wheel_track} ${wheel_front_rear_radius}" />
   </joint>
-  <link name="lifting_platform_base">
+  <link name="basic_platform">
     <inertial>
       <origin xyz="0. 0. 0." />
@@ -218,13 +212,13 @@
     </inertial>
     <visual>
-      <origin rpy="0. 0. ${pi/2}" xyz="0. 0. ${base_link_height + lift_base_offset}"/>
-      <geometry>
-        <mesh filename="../meshes/Platform_B.stl" scale="1.0 1.0 1.0" />
+      <origin rpy="0. 0. ${pi/2}" xyz="0. 0. ${basic_platform_offset}"/>
+      <geometry>
+        <mesh filename="../meshes/Platform_A.stl" scale="1.0 1.0 1.0" />
       </geometry>
     </visual>
     <collision>=
-      <origin rpy="0. 0. ${pi/2}" xyz="0. 0. ${base_link_height + lift_base_offset + lift_base_collider_offset}"/>
-      <geometry>
-        <box size="${lift_base_width} ${lift_base_length} ${lift_base_height}" />
+      <origin rpy="0. 0. ${pi/2}" xyz="0. 0. ${basic_platform_offset + basic_platform_collider_offset}"/>
+      <geometry>
+        <box size="${basic_platform_width} ${basic_platform_length} ${basic_platform_height}" />
       </geometry>
     </collision>
@@ -232,50 +226,6 @@
   <joint name="platform_base_joint" type="fixed">
     <parent link="base_link" />
-    <child link="lifting_platform_base" />
+    <child link="basic_platform" />
     <origin rpy="0. 0. 0." xyz="0. 0. 0." />
-  </joint>
-  <link name="lift_module">
-    <inertial>
-      <origin xyz="0. 0. 0." />
-      <mass value="15" />
-      <inertia ixx="1." ixy="0." ixz="0." iyy="1." iyz="0." izz="1."/>
-    </inertial>
-    <visual>
-      <origin rpy="0. 0. ${pi/2}" xyz="0. 0. 0."/>
-      <geometry>
-        <mesh filename="../meshes/lift.stl" scale="1.0 1.0 1.0" />
-      </geometry>
-    </visual>
-  </link>
-  <joint name="lift_module_joint" type="fixed">
-    <parent link="base_link" />
-    <child link="lift_module" />
-    <origin rpy="0. 0. 0." xyz="0. 0. ${base_link_height + lift_base_offset + lift_module_offset}" />
-  </joint>
-  <link name="lift_upper">
-    <inertial>
-      <origin xyz="0. 0. 0." />
-      <mass value="15" />
-      <inertia ixx="1." ixy="0." ixz="0." iyy="1." iyz="0." izz="1."/>
-    </inertial>
-    <visual>
-      <origin rpy="0. 0. ${pi/2}" xyz="0. 0. ${base_link_box_height + lift_module_height}"/>
-      <geometry>
-        <mesh filename="../meshes/lift_upper.stl" scale="1.0 1.0 1.0" />
-      </geometry>
-    </visual>
-    <collision>
-      <origin rpy="0. 0. ${pi/2}" xyz="0. 0. ${base_link_box_height + lift_module_height}"/>
-      <geometry>
-        <box size="${lift_upper_width} ${lift_upper_length} ${lift_upper_height}" />
-      </geometry>
-    </collision>
-  </link>
-  <joint name="lift_upper_joint" type="prismatic">
-    <parent link="base_link" />
-    <child link="lift_upper" />
-    <axis xyz="0. 0. 1." />
-    <origin rpy="0. 0. 0." xyz="0. 0. 0." />
-    <limit lower="0.0" upper="${upper_lift_limit}" effort="0.0" velocity="0.0"/>
   </joint>
   <link name="lidar_F" />
