Commit message: Add lift to otto1500 urdf
Signed-off-by: Anna Faferek <anna.faferek@robotec.ai>

File: ros2_ws/src/OTTO1500_Description/urdf/OTTO1500.urdf.xacro (robot description, xacro)
@@ -3,5 +3,6 @@
   <xacro:property name="base_link_length" value="1.83" />
   <xacro:property name="base_link_width" value="1.29" />
-  <xacro:property name="base_link_height" value="0.406" />
+  <xacro:property name="base_link_height" value="0.32" />
+  <xacro:property name="base_link_box_height" value=".391179" />
   <xacro:property name="ground_clearence" value="0.1" />
   <xacro:property name="wheel_axis_front" value="0.601175" />
@@ -12,4 +13,9 @@
   <xacro:property name="wheel_center_radius" value="0.147" />
   <xacro:property name="wheel_center_length" value="0.1" />
+  <xacro:property name="upper_lift_limit" value="0.3" />
+  <xacro:property name="lift_module_height" value="0.15" />
+  <xacro:property name="camera_height" value="0.22" />
+  <xacro:property name="camera_center_offset" value="0.51" />
+  <xacro:property name="lidar_height" value="0.1" />
   <link name="base_link">
     <inertial>
@@ -182,3 +188,107 @@
     <origin rpy="0. 0. 0." xyz="${wheel_axis_rear} ${-wheel_track} ${wheel_front_rear_radius}" />
   </joint>
+  <link name="lifting_platform_base">
+    <inertial>
+      <origin xyz="0. 0. 0." />
+      <mass value="15" />
+      <inertia ixx="1." ixy="0." ixz="0." iyy="1." iyz="0." izz="1."/>
+    </inertial>
+    <visual>
+      <origin rpy="0. 0. ${pi/2}" xyz="0. 0. 0."/>
+      <geometry>
+        <mesh filename="../meshes/Platform_B.stl" scale="1.0 1.0 1.0" />
+      </geometry>
+    </visual>
+    <collision>=
+      <origin rpy="0. 0. ${pi/2}" xyz="0. 0. ${base_link_height + ground_clearence}"/>
+      <geometry>
+        <box size="1. 1.35 0.14" />
+      </geometry>
+    </collision>
+  </link>
+  <joint name="platform_base_joint" type="fixed">
+    <parent link="base_link" />
+    <child link="lifting_platform_base" />
+    <origin rpy="0. 0. 0." xyz="0. 0. 0." />
+  </joint>
+  <link name="lift_module">
+    <inertial>
+      <origin xyz="0. 0. 0." />
+      <mass value="15" />
+      <inertia ixx="1." ixy="0." ixz="0." iyy="1." iyz="0." izz="1."/>
+    </inertial>
+    <visual>
+      <origin rpy="0. 0. ${pi/2}" xyz="0. 0. 0."/>
+      <geometry>
+        <mesh filename="../meshes/lift.stl" scale="1.0 1.0 1.0" />
+      </geometry>
+    </visual>
+  </link>
+  <joint name="lift_module_joint" type="prismatic">
+    <parent link="lifting_platform_base" />
+    <child link="lift_module" />
+    <axis xyz="0. 0. 1." />
+    <origin rpy="0. 0. 0." xyz="0. 0. 0." />
+    <limit lower="0.0" upper="${upper_lift_limit}" effort="0.0" velocity="0.0"/>
+  </joint>
+  <link name="lift_upper">
+    <inertial>
+      <origin xyz="0. 0. 0." />
+      <mass value="15" />
+      <inertia ixx="1." ixy="0." ixz="0." iyy="1." iyz="0." izz="1."/>
+    </inertial>
+    <visual>
+      <origin rpy="0. 0. ${pi/2}" xyz="0. 0. 0."/>
+      <geometry>
+        <mesh filename="../meshes/lift_upper.stl" scale="1.0 1.0 1.0" />
+      </geometry>
+    </visual>
+    <collision>
+      <origin rpy="0. 0. ${pi/2}" xyz="0. 0. ${base_link_box_height + lift_module_height}"/>
+      <geometry>
+        <box size="0.5 1.2 0.02" />
+      </geometry>
+    </collision>
+  </link>
+  <joint name="lift_upper_joint" type="fixed">
+    <parent link="lift_module" />
+    <child link="lift_upper" />
+    <origin rpy="0. 0. 0." xyz="0. 0. 0." />
+  </joint>
+  <link name="lidar_F" />
+  <joint name="lidar_F_joint" type="fixed">
+    <parent link="base_link" />
+    <child link="lidar_F" />
+    <origin rpy="0. 0. 0." xyz="${base_link_length * 0.47} ${base_link_width * 0.47} ${lidar_height}" />
+  </joint>
+  <link name="lidar_R" />
+  <joint name="lidar_R_joint" type="fixed">
+    <parent link="base_link" />
+    <child link="lidar_R" />
+    <origin rpy="0. 0. 0." xyz="${-base_link_length * 0.47} ${-base_link_width * 0.47} ${lidar_height}" />
+  </joint>
+  <link name="camera_FL" />
+  <joint name="camera_FL_joint" type="fixed">
+    <parent link="base_link" />
+    <child link="camera_FL" />
+    <origin rpy="0. 0. 0." xyz="${base_link_length / 2} ${camera_center_offset} ${camera_height}" />
+  </joint>
+  <link name="camera_FR" />
+  <joint name="camera_FR_joint" type="fixed">
+    <parent link="base_link" />
+    <child link="camera_FR" />
+    <origin rpy="0. 0. 0." xyz="${base_link_length / 2} ${-camera_center_offset} ${camera_height}" />
+  </joint>
+  <link name="camera_RL" />
+  <joint name="camera_RL_joint" type="fixed">
+    <parent link="base_link" />
+    <child link="camera_RL" />
+    <origin rpy="0. 0. 0." xyz="${-base_link_length / 2} ${camera_center_offset} ${camera_height}" />
+  </joint>
+  <link name="camera_RR" />
+  <joint name="camera_RR_joint" type="fixed">
+    <parent link="base_link" />
+    <child link="camera_RR" />
+    <origin rpy="0. 0. 0." xyz="${-base_link_length / 2} ${-camera_center_offset} ${camera_height}" />
+  </joint>
 </robot>

Commit message: Revert "Change colliders in urdf"
This reverts commit 692a444e1e1d0f3ecee9630aa5068b1dc900ee6b.

File: ros2_ws/src/OTTO1500_Description/urdf/OTTO1500.urdf.xacro (robot description, xacro)
@@ -5,4 +5,5 @@
   <xacro:property name="base_link_height" value="0.32" />
   <xacro:property name="base_link_box_height" value=".391179" />
+  <xacro:property name="ground_clearence" value="0.1" />
   <xacro:property name="wheel_axis_front" value="0.601175" />
   <xacro:property name="wheel_axis_rear" value="-0.601175" />
@@ -38,23 +39,8 @@
       </geometry>
     </visual>
-    <!-- bottom collider box -->
-    <collision>
-      <origin rpy="0. 0. ${pi/2}" xyz="0. 0. 0.049"/>
-      <geometry>
-        <box size="${base_link_width} ${base_link_length} 0.05" />
-      </geometry>
-    </collision>
-    <!-- center collider box -->
-    <collision>
-      <origin rpy="0. 0. ${pi/2}" xyz="0. 0. 0.114"/>
-      <geometry>
-        <box size="1.135 1.663 0.079" />
-      </geometry>
-    </collision>
-    <!-- top collider box -->
-    <collision>
-      <origin rpy="0. 0. ${pi/2}" xyz="0. 0. 0.248"/>
-      <geometry>
-        <box size="${base_link_width} ${base_link_length} 0.187" />
+    <collision>
+      <origin rpy="0. 0. ${pi/2}" xyz="0. 0. ${base_link_height* (0.5 + ground_clearence/2)}"/>
+      <geometry>
+        <box size="${base_link_width} ${base_link_length} ${base_link_height}" />
       </geometry>
     </collision>

File: ros2_ws/src/OTTO1500_Description/urdf/OTTO1500_basic_platform.urdf.xacro (robot description, xacro)
@@ -5,4 +5,5 @@
   <xacro:property name="base_link_height" value="0.32" />
   <xacro:property name="base_link_box_height" value=".391179" />
+  <xacro:property name="ground_clearence" value="0.1" />
   <xacro:property name="wheel_axis_front" value="0.601175" />
   <xacro:property name="wheel_axis_rear" value="-0.601175" />
@@ -32,23 +33,8 @@
       </geometry>
     </visual>
-    <!-- bottom collider box -->
-    <collision>
-      <origin rpy="0. 0. ${pi/2}" xyz="0. 0. 0.049"/>
-      <geometry>
-        <box size="${base_link_width} ${base_link_length} 0.05" />
-      </geometry>
-    </collision>
-    <!-- center collider box -->
-    <collision>
-      <origin rpy="0. 0. ${pi/2}" xyz="0. 0. 0.114"/>
-      <geometry>
-        <box size="1.135 1.663 0.079" />
-      </geometry>
-    </collision>
-    <!-- top collider box -->
-    <collision>
-      <origin rpy="0. 0. ${pi/2}" xyz="0. 0. 0.248"/>
-      <geometry>
-        <box size="${base_link_width} ${base_link_length} 0.187" />
+    <collision>
+      <origin rpy="0. 0. ${pi/2}" xyz="0. 0. ${base_link_height* (0.5 + ground_clearence/2)}"/>
+      <geometry>
+        <box size="${base_link_width} ${base_link_length} ${base_link_height}" />
       </geometry>
     </collision>

Commit message: fixes after review

File: ros2_ws/src/OTTO1500_Description/urdf/OTTO1500.urdf.xacro (robot description, xacro)
@@ -5,5 +5,4 @@
   <xacro:property name="base_link_height" value="0.32" />
   <xacro:property name="base_link_box_height" value=".391179" />
-  <xacro:property name="ground_clearence" value="0.1" />
   <xacro:property name="wheel_axis_front" value="0.601175" />
   <xacro:property name="wheel_axis_rear" value="-0.601175" />
@@ -39,8 +38,23 @@
       </geometry>
     </visual>
-    <collision>
-      <origin rpy="0. 0. ${pi/2}" xyz="0. 0. ${base_link_height* (0.5 + ground_clearence/2)}"/>
-      <geometry>
-        <box size="${base_link_width} ${base_link_length} ${base_link_height}" />
+    <!-- bottom collider box -->
+    <collision>
+      <origin rpy="0. 0. ${pi/2}" xyz="0. 0. 0.049"/>
+      <geometry>
+        <box size="${base_link_width} ${base_link_length} 0.05" />
+      </geometry>
+    </collision>
+    <!-- center collider box -->
+    <collision>
+      <origin rpy="0. 0. ${pi/2}" xyz="0. 0. 0.114"/>
+      <geometry>
+        <box size="1.135 1.663 0.079" />
+      </geometry>
+    </collision>
+    <!-- top collider box -->
+    <collision>
+      <origin rpy="0. 0. ${pi/2}" xyz="0. 0. 0.248"/>
+      <geometry>
+        <box size="${base_link_width} ${base_link_length} 0.187" />
       </geometry>
     </collision>

File: ros2_ws/src/OTTO1500_Description/urdf/OTTO1500_basic_platform.urdf.xacro (robot description, xacro)
@@ -5,5 +5,4 @@
   <xacro:property name="base_link_height" value="0.32" />
   <xacro:property name="base_link_box_height" value=".391179" />
-  <xacro:property name="ground_clearence" value="0.1" />
   <xacro:property name="wheel_axis_front" value="0.601175" />
   <xacro:property name="wheel_axis_rear" value="-0.601175" />
@@ -33,8 +32,23 @@
       </geometry>
     </visual>
-    <collision>
-      <origin rpy="0. 0. ${pi/2}" xyz="0. 0. ${base_link_height* (0.5 + ground_clearence/2)}"/>
-      <geometry>
-        <box size="${base_link_width} ${base_link_length} ${base_link_height}" />
+    <!-- bottom collider box -->
+    <collision>
+      <origin rpy="0. 0. ${pi/2}" xyz="0. 0. 0.049"/>
+      <geometry>
+        <box size="${base_link_width} ${base_link_length} 0.05" />
+      </geometry>
+    </collision>
+    <!-- center collider box -->
+    <collision>
+      <origin rpy="0. 0. ${pi/2}" xyz="0. 0. 0.114"/>
+      <geometry>
+        <box size="1.135 1.663 0.079" />
+      </geometry>
+    </collision>
+    <!-- top collider box -->
+    <collision>
+      <origin rpy="0. 0. ${pi/2}" xyz="0. 0. 0.248"/>
+      <geometry>
+        <box size="${base_link_width} ${base_link_length} 0.187" />
       </geometry>
     </collision>
